File: KiCad_project_current/DesignLab_project_PS_MC_SS.kicad_pcb (KiCad board)
At the start: 2 copper layers, 133.5 x 89 mm, 61 parts, among them J1 Conn_01x09, J2 USB_B_Micro, J3 Barrel_Jack, J4 Conn_02x08_Odd_Even, SW1 SW_Push, SW2 SW_Push, SW3 SW_Push, SW4 SW_Push, SW5 SW_Push, U1 ATmega328P-P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

Commit message: Current version of KiCad project
Parts:
- moved J2 120.5 mm to (241.3, 62.5), turned to 90 degrees
- moved C16 98.4 mm to (227.0, 72.0), turned to 90 degrees
- moved C18 98.4 mm to (237.5, 72.1)
- moved C17 98.3 mm to (232.5, 72.1)
- moved U2 86.7 mm to (226.0, 61.9)
- moved C3 70.8 mm to (158.5, 62.5)
- moved R1 70.8 mm to (158.5, 49.5)
- moved SW1 70.8 mm to (158.5, 56.0)
- moved J3 56.5 mm to (234.0, 114.5)
- moved R13 40.2 mm to (205.0, 116.5), turned to 180 degrees
- moved R12 40.2 mm to (205.0, 109.0), turned to 180 degrees
- moved C11 36.9 mm to (213.5, 108.5), turned to 180 degrees
- moved R11 35.2 mm to (205.0, 103.5), turned to 180 degrees
- moved C12 34.6 mm to (213.5, 113.5), turned to 180 degrees
- moved C10 34.2 mm to (217.5, 101.3)
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Routing:
- net RESET: track 180.6 -> 45.2 mm, vias 2 -> 0
- net +3.3V: track 308.8 -> 197.8 mm, vias 3 -> 5
- net GND: track 693.0 -> 586.0 mm, vias 20 -> 234
- net PB1: track 18.5 -> 52.3 mm
- net PD2: track 64.9 -> 37.4 mm, vias 2 -> 0
- net TX/PD1: track 93.5 -> 119.5 mm, vias 4 -> 2
- net SCK: track 46.3 -> 21.3 mm, vias 2 -> 0
- net PD4: track 82.2 -> 61.0 mm, vias 0 -> 2
- net PC4: track 40.7 -> 24.5 mm, vias 2 -> 0
- net PD3: track 76.4 -> 60.5 mm
- net PD7: track 77.6 -> 62.5 mm, vias 2 -> 0
- net PC5: track 31.9 -> 17.1 mm
- net PD5: track 49.1 -> 34.6 mm
- net PD6: track 63.7 -> 49.7 mm
- net PB2: track 62.5 -> 75.4 mm, vias 2 -> 0
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Other:
- board size 133.5 x 89 mm -> 120.4 x 91.9 mm

Commit message: Current version of KiCad project
Parts:
- moved R21 20.4 mm to (149.8, 85.1), turned to 180 degrees
- moved C16 14.9 mm to (230.7, 57.6), turned to 0 degrees
- moved R20 12.4 mm to (149.8, 80.0)
- moved R1 11.7 mm to (158.2, 61.2)
- moved C3 10.8 mm to (169.0, 60.0), turned to 90 degrees
- moved C11 8.81 mm to (205.0, 106.2)
- moved C17 8.58 mm to (240.1, 68.1), turned to 0 degrees
- moved C12 8.55 mm to (205.0, 113.1)
- moved C9 6.67 mm to (194.3, 72.9)
- moved R3 5.80 mm to (185.1, 57.4), turned to 90 degrees
- moved C8 5.64 mm to (229.2, 95.1)
- moved R19 5.03 mm to (149.8, 73.6)
- moved R16 3.63 mm to (149.8, 70.0)
- moved R14 3.43 mm to (149.8, 67.2)
- moved U2 3.14 mm to (229.0, 63.0), turned to -90 degrees
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Routing:
- net GND: track 586.0 -> 511.6 mm, vias 234 -> 58
- net +5V: track 482.4 -> 408.6 mm, vias 6 -> 2
- net +3.3V: track 197.8 -> 165.3 mm, vias 5 -> 2
- net PD7: track 62.5 -> 38.4 mm
- net Net-(U6-G): track 4.16 -> 18.6 mm
- net PD6: track 49.7 -> 35.5 mm
- net Net-(U2-V3): track 16.0 -> 2.90 mm
- net Net-(U6-DP): track 3.95 -> 16.4 mm
- net PD3: track 60.5 -> 52.0 mm
- net RESET: track 45.2 -> 36.8 mm
- net AREF: track 9.83 -> 3.25 mm
- net RX/PD0: track 113.6 -> 118.7 mm
- net TX/PD1: track 119.5 -> 124.0 mm
- net PD4: track 61.0 -> 56.6 mm
- net PC4: track 24.5 -> 20.7 mm
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
Commit message: Final version of the KiCad project
Parts:
- C1, C10, C11, C12, C13, C14, C16, C18, C2, C3, C5, C7, C8, C9: footprint Capacitor_SMD:C_0805_2012Metric_Pad1.18x1.45mm_HandSolder -> Capacitor_SMD:C_0603_1608Metric
- C17, C6: footprint Capacitor_SMD:C_0805_2012Metric_Pad1.18x1.45mm_HandSolder -> Capacitor_SMD:CP_Elec_4x3
- D2, D3, D4, D5, D6, D7: footprint LED_SMD:LED_0201_0603Metric_Pad0.64x0.40mm_HandSolder -> LED_SMD:LED_0603_1608Metric
- J4: footprint Connector_PinHeader_2.54mm:PinHeader_2x08_P2.54mm_Vertical_SMD -> Connector_PinHeader_2.54mm:PinHeader_2x08_P2.54mm_Vertical
- R4, R5, R6, R7, R8, R9: value 1kOhm -> 1k
- moved R10 57.2 mm to (148.5, 108.2), turned to -90 degrees
- moved R11 52.7 mm to (152.5, 108.2), turned to -90 degrees
- moved U2 52.2 mm to (179.0, 78.0), turned to 180 degrees
- moved C16 50.7 mm to (185.5, 80.7), turned to -90 degrees
- moved C11 49.8 mm to (155.2, 108.2), turned to -90 degrees
- moved C17 46.7 mm to (195.8, 82.9)
- moved R12 46.5 mm to (158.5, 108.2), turned to -90 degrees
- moved C18 46.1 mm to (196.8, 88.4)
- moved C6 46.0 mm to (177.9, 105.4)
- moved C10 45.7 mm to (171.9, 104.0)
- moved U7 45.7 mm to (174.4, 93.2)
- moved U5 43.3 mm to (191.8, 102.2)
- moved C7 43.3 mm to (193.3, 108.4)
- moved C8 43.3 mm to (187.0, 105.0)
- moved C12 43.2 mm to (162.1, 108.2), turned to -90 degrees
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Routing:
- net GND: track 511.6 -> 459.7 mm, vias 58 -> 57
- net +3.3V: track 165.3 -> 126.9 mm, vias 2 -> 3
- net PB2: track 75.4 -> 91.0 mm, vias 0 -> 1
- net PB3: track 63.3 -> 77.8 mm, vias 2 -> 1
- net RX/PD0: track 118.7 -> 109.5 mm
- net PB5: track 41.2 -> 49.8 mm
- net PD3: track 52.0 -> 59.0 mm
- net TX/PD1: track 124.0 -> 117.4 mm
- net MISO: track 20.1 -> 13.7 mm
- net SCK: track 21.3 -> 15.1 mm
- net PB4: track 57.9 -> 64.1 mm, vias 0 -> 1
- net D+: track 13.0 -> 18.7 mm, vias 0 -> 2
- net MOSI: track 23.4 -> 19.6 mm, vias 0 -> 1
- net +5V: track 408.6 -> 405.1 mm
- net D-: track 14.5 -> 17.7 mm
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Other:
- board size 120.4 x 91.9 mm -> 111.9 x 80.9 mm
