File: KiCad_project_current/DesignLab_project_PS_MC_SS.kicad_sch (KiCad schematic)
At the start: 61 parts, among them J1 Conn_01x09, J2 USB_B_Micro, J3 Barrel_Jack, J4 Conn_02x08_Odd_Even, SW1 SW_Push, SW2 SW_Push, SW3 SW_Push, SW4 SW_Push, SW5 SW_Push, U1 ATmega328P-P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

Commit message: Final version of the KiCad project
Parts:
- C1, C10, C11, C12, C13, C14, C16, C18, C2, C3, C5, C7, C8, C9: footprint Capacitor_SMD:C_0805_2012Metric_Pad1.18x1.45mm_HandSolder -> Capacitor_SMD:C_0603_1608Metric
- C17: footprint Capacitor_SMD:C_0805_2012Metric_Pad1.18x1.45mm_HandSolder -> Capacitor_SMD:CP_Elec_4x3; symbol Device:C -> Device:C_Polarized
- C6: footprint Capacitor_SMD:C_0805_2012Metric_Pad1.18x1.45mm_HandSolder -> Capacitor_SMD:CP_Elec_4x3
- D2, D3, D4, D5, D6, D7: footprint LED_SMD:LED_0201_0603Metric_Pad0.64x0.40mm_HandSolder -> LED_SMD:LED_0603_1608Metric
- J4: footprint Connector_PinHeader_2.54mm:PinHeader_2x08_P2.54mm_Vertical_SMD -> Connector_PinHeader_2.54mm:PinHeader_2x08_P2.54mm_Vertical
- R4, R5, R6, R7, R8, R9: value 1kOhm -> 1k
Other:
- note added: "Diodes"
- note added: "Switches"
- note added: "Temperature & pressure sensor"
- note added: "Temperature sensor"
- note added: "USB implementation"
- note removed: "Diodes and switches"
- note removed: "SENSORS"
- note removed: "USB implenetation"
- moved on the sheet: C10, C11, C12, C13, C14, C16, C18, C3, C6, C9, D2, D3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
